File: eagle/LME49600_HPA.brd (EAGLE design)
At the start: 93.7 x 71.1 mm, 47 parts, among them IC1 OPA2134P, IC2 OPA2134P, P1 POLYSWITCH, P2 POLYSWITCH

Commit message: Update: Board design
Parts:
- moved C7 14.8 mm to (40.6, 59.7)
- moved C6 13.7 mm to (40.6, 47.0), turned to 270 degrees
- moved U$1 13.0 mm to (53.3, 53.3)
- moved R1 11.5 mm to (10.2, 64.8), turned to 90 degrees
- moved C8 10.5 mm to (25.4, 45.7)
- moved C2 10.5 mm to (27.9, 54.6)
- moved C3 10.5 mm to (10.2, 54.6)
- moved C9 10.5 mm to (10.2, 45.7)
- moved IC1 10.5 mm to (19.1, 54.6)
- moved R2 10.5 mm to (24.1, 61.0)
- moved R3 10.5 mm to (24.1, 63.5)
- moved R4 10.5 mm to (17.8, 44.5)
- moved R6 10.5 mm to (20.3, 44.5)
- moved R5 10.5 mm to (15.2, 44.5)
- moved R13 8.03 mm to (69.8, 38.1)
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Routing:
- net AGND: track 167.5 -> 418.5 mm
- net V+: track 29.0 -> 171.7 mm
- net V-: track 56.6 -> 198.6 mm
- net N$13: track 0.00 -> 80.8 mm
- net N$4: track 0.00 -> 63.5 mm
- net N$14: track 63.1 -> 91.0 mm
- net N$3: track 38.7 -> 63.5 mm
- net N$5: track 0.00 -> 23.9 mm
- net N$16: track 0.00 -> 16.3 mm
- net N$9: track 0.00 -> 15.2 mm
- net PW+: track 0.00 -> 13.1 mm
- net PW-: track 0.00 -> 13.0 mm
- net N$19: track 0.00 -> 7.62 mm
- net N$17: track 0.00 -> 7.62 mm
- net N$10: track 0.00 -> 7.62 mm
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
Commit message: Update: Board design
Parts:
- C11, C20: value (none) -> 2.2uF
- R1, R12: value 1.2k -> 47k
- moved C16 5.08 mm to (30.5, 10.2)
- moved C8 5.08 mm to (30.5, 45.7)
- moved R2 2.54 mm to (26.7, 61.0)
- moved R3 2.54 mm to (26.7, 63.5)
- moved R7 2.54 mm to (26.7, 25.4)
- moved R8 2.54 mm to (26.7, 27.9)
- moved C11 2.54 mm to (17.8, 63.5)
- moved C20 2.54 mm to (17.8, 27.9)
- moved R10 2.54 mm to (17.8, 8.89)
- moved R5 2.54 mm to (17.8, 44.5)
- moved C1 2.54 mm to (85.1, 58.4)
- moved C12 2.54 mm to (30.5, 19.1)
- moved C13 2.54 mm to (12.7, 19.1)
- moved C17 2.54 mm to (12.7, 10.2)
- moved C2 2.54 mm to (30.5, 54.6)
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Routing:
- net AGND: track 418.5 -> 455.4 mm
- net V+: track 171.7 -> 151.9 mm
- net V-: track 198.6 -> 182.0 mm
- net N$14: track 91.0 -> 84.4 mm
- net N$13: track 80.8 -> 76.8 mm
- net PW+: track 13.1 -> 9.40 mm
- net PW-: track 13.0 -> 9.40 mm
- net N$7: track 23.9 -> 21.4 mm
- net N$12: track 7.62 -> 10.2 mm
- net N$11: track 7.62 -> 10.2 mm
- net N$15: track 7.62 -> 10.2 mm
- net N$1: track 7.62 -> 10.2 mm
- net N$5: track 23.9 -> 21.4 mm
- net N$9: track 15.2 -> 16.3 mm
- net N$6: track 15.2 -> 16.3 mm

Commit message: Completed Soldering
Parts:
- removed C11, C20: 2.2uF, rcl:C050-055X075
- removed JP5: OUT, pinhead:1X02
- removed P1, P2: POLYSWITCH, mylib2:POLYSWITCH
- removed PWR: (no value), con-wago-508:W237-4P
- removed R1, R12: 47k, rcl:0207/7
- added JP3: IN, pinhead:1X02
- added JP6: PWR-, pinhead:1X02
- added JP7: PWR+, pinhead:1X02
- JP4: value IN -> OUT
- moved JP4 41.0 mm to (45.7, 31.8), turned to 90 degrees
- moved R13 5.08 mm to (74.9, 38.1)
- moved R14 5.08 mm to (74.9, 33.0)
Connections:
- removed net N$16: C20.1, IC2.3, R12.2
- removed net N$2: C11.1, IC1.3, R1.2
- removed net PW+: P1.2, PWR.1
- removed net PW-: P2.2, PWR.4
- net AGND: now also JP3.2, JP6.1, JP7.2; no longer JP5.2, PWR.2, PWR.3, R1.1, R12.1
- net N$1: now also IC1.3; no longer C11.2
- net N$13: now also JP4.1; no longer JP5.1
- net N$15: now also IC2.3, JP3.1; no longer C20.2, JP4.1
- net V+: now also JP7.1; no longer P1.1
- net V-: now also JP6.2; no longer P2.1
Routing:
- net AGND: track 455.4 -> 435.9 mm
- net V+: track 151.9 -> 170.7 mm
- net N$16: track 16.3 -> 0.00 mm
- net N$2: track 16.3 -> 0.00 mm
- net V-: track 182.0 -> 192.6 mm
- net PW-: track 9.40 -> 0.00 mm
- net PW+: track 9.40 -> 0.00 mm
- net N$15: track 10.2 -> 18.8 mm
- net N$1: track 10.2 -> 18.8 mm
- net N$19: track 7.62 -> 2.54 mm
- net N$17: track 7.62 -> 2.54 mm
