File: eagle/LME49600_HPA.sch (EAGLE design)
At the start: 47 parts, among them IC1 OPA2134P, IC2 OPA2134P, P1 POLYSWITCH, P2 POLYSWITCH

Commit message: Completed Soldering
Parts:
- removed C11, C20: 2.2uF, rcl:C-EU050-055X075
- removed JP5: OUT, pinhead:PINHD-1X2
- removed P1, P2: POLYSWITCH, mylib2:POLYSWITCH
- removed PWR: (no value), con-wago-508:W237-04P
- removed R1, R12: 47k, rcl:R-EU_0207/7
- added JP3: IN, pinhead:PINHD-1X2
- added JP6: PWR-, pinhead:PINHD-1X2
- added JP7: PWR+, pinhead:PINHD-1X2
- JP4: value IN -> OUT
Connections:
- removed net N$16: C20.1, IC2A.+IN, R12.2
- removed net N$2: C11.1, IC1A.+IN, R1.2
- removed net PW+: P1.2, PWR-1.KL
- removed net PW-: P2.2, PWR-4.KL
- net AGND: now also JP3.2, JP6.1, JP7.2; no longer JP5.2, PWR-2.KL, PWR-3.KL, R1.1, R12.1
- net N$1: now also IC1A.+IN; no longer C11.2
- net N$13: now also JP4.1; no longer JP5.1
- net N$15: now also IC2A.+IN, JP3.1; no longer C20.2, JP4.1
- net V+: now also JP7.1; no longer P1.1
- net V-: now also JP6.2; no longer P2.1
Other:
- note removed: "R1, R12, C11, C22はピンソケットで実装"
- moved on the sheet: JP4
